File: holocubic.kicad_sch (KiCad schematic)
At the start: 11 parts

Commit message: update
Parts:
- added AE?: (no value), symbol Device:Antenna_Shield
- added C? (x2): (no value), Capacitor_SMD:C_0402_1005Metric, symbol Device:C
- added C?: (no value), symbol Device:C
- added C?: 10uf, Capacitor_SMD:C_0603_1608Metric, symbol Device:C
- added J?: (no value), symbol Connector_Generic:Conn_01x08
- added L?: (no value), symbol Device:L
- added TP? (x5): TestPoint, symbol Connector:TestPoint
- added TP?: (no value), symbol Connector:TestPoint
- added U?: (no value), symbol Audio:WM8731CSEFL
- added U?: (no value), symbol Regulator_Linear:AMS1117CD-3.3
- C? (x3): value (none) -> 0.1uf; footprint (none) -> Capacitor_SMD:C_0402_1005Metric
- C? (x2): value (none) -> 10pf; footprint (none) -> Capacitor_SMD:C_0402_1005Metric
- C? (x2): value (none) -> 1uf; footprint (none) -> Capacitor_SMD:C_0402_1005Metric
- R?: value (none) -> R; footprint (none) -> Resistor_SMD:R_0402_1005Metric
- U?: value (none) -> ESP32-S3; footprint (none) -> Package_DFN_QFN:QFN-56-1EP_7x7mm_P0.4mm_EP5.6x5.6mm
- Y?: value (none) -> 40MHz
Connections:
- net +3V3: now also C?.1, TP?.1, U?.2 (VO)
- net GND: now also AE?.2 (Shield), C?.2, C?.2, C?.2, C?.2, TP?.1, U?.1 (GND)
- net LNA: now also C?.1, L?.1
- net RST: now also TP?.1
- net +5V: now reaches J?.A4 (VBUS), J?.A9 (VBUS), J?.B4 (VBUS), J?.B9 (VBUS)
- net +5V: now also C?.1, U?.3 (VI)
- net at U?.10 (GPIO5/ADC1_CH4): now also J?.5 (Pin_5)
- net at U?.11 (GPIO6/ADC1_CH5): now also J?.6 (Pin_6)
- net at U?.12 (GPIO7/ADC1_CH6): now also J?.7 (Pin_7)
- net at U?.13 (GPIO8/ADC1_CH7): now also J?.8 (Pin_8)
- net TX0: now reaches U?.49 (U0TXD/PROG/GPIO43)
- net TX0: now also TP?.1
- net IO0: now reaches U?.5 (GPIO0/BOOT)
- net IO0: now also TP?.1
- net RX0: now reaches U?.50 (U0RXD/PROG/GPIO44)
- net RX0: now also TP?.1
- net at U?.6 (GPIO1/ADC1_CH0): now also J?.1 (Pin_1)
- net at U?.7 (GPIO2/ADC1_CH1): now also J?.2 (Pin_2)
- net at U?.8 (GPIO3/ADC1_CH2): now also J?.3 (Pin_3)
- net at U?.9 (GPIO4/ADC1_CH3): now also J?.4 (Pin_4)
- new net: AE?.1 (A), C?.1, L?.2
- new net: U?.19 (AGND), U?.29 (AGND)
Other:
- title: (none) -> main-board
- moved on the sheet: C?, R?
