File: hardware/holocubic.kicad_sch (KiCad schematic)
At the start: 26 parts

Commit message: hw: update
Parts:
- removed U?: (no value), symbol Audio:WM8731CSEFL
- added C? (x10): (no value), symbol Device:C
- added J?: Speaker, symbol Connector_Generic:Conn_01x02
- added MK?: Microphone_MEMS, symbol misc:Microphone_MEMS
- added R? (x3): (no value), symbol Device:R
- added U?: WM8978, Package_DFN_QFN:QFN-32-1EP_5x5mm_P0.5mm_EP3.3x3.3mm, symbol misc:WM8978
- C? (x3): value 0.1uf -> (none); footprint Capacitor_SMD:C_0402_1005Metric -> (none)
- C? (x2): footprint Capacitor_SMD:C_0402_1005Metric -> (none)
- C? (x2): value 10pf -> (none); footprint Capacitor_SMD:C_0402_1005Metric -> (none)
- C?: value 10uf -> (none); footprint Capacitor_SMD:C_0603_1608Metric -> (none)
- C? (x2): value 1uf -> (none); footprint Capacitor_SMD:C_0402_1005Metric -> (none)
- R?: value R -> (none); footprint Resistor_SMD:R_0402_1005Metric -> (none)
- TP? (x5): value TestPoint -> (none)
- U?: value ESP32-S3 -> (none); footprint Package_DFN_QFN:QFN-56-1EP_7x7mm_P0.4mm_EP5.6x5.6mm -> (none)
- Y?: value 40MHz -> (none)
Connections:
- net +3V3: now also J?.7 (Pin_7), C?.1, C?.2, C?.2, U?.13 (DCVDD), U?.14 (DBVDD), U?.26 (SPKVDD), U?.31 (AVDD)
- net GND: now also J?.8 (Pin_8), C?.1, C?.1, C?.1, C?.1, C?.1, C?.2, C?.2, C?.2, MK?.2 (GND), MK?.3 (GND), R?.1, R?.2, R?.2, U?.12 (DGND), U?.18 (MODE), U?.24 (SPKGND), U?.28 (AGND), U?.33 (GNDPAD)
- net at J?.A5 (CC1): now also R?.1
- net at J?.B5 (CC2): now also R?.1
- net at U?.10 (GPIO5/ADC1_CH4): no longer J?.5 (Pin_5)
- net at U?.11 (GPIO6/ADC1_CH5): no longer J?.6 (Pin_6)
- net at U?.12 (GPIO7/ADC1_CH6): no longer J?.7 (Pin_7)
- net at U?.13 (GPIO8/ADC1_CH7): no longer J?.8 (Pin_8)
- net LCD_MOSI: now reaches U?.15 (GPIO10/ADC1_CH9)
- net LCD_MOSI: now also J?.1 (Pin_1)
- net LCD_SCK: now reaches U?.16 (GPIO11/ADC2_CH0)
- net LCD_SCK: now also J?.2 (Pin_2)
- net LCD_CS: now reaches U?.17 (GPIO12/ADC2_CH1)
- net LCD_CS: now also J?.3 (Pin_3)
- net LCD_DC: now reaches U?.18 (GPIO13/ADC2_CH2)
- net LCD_DC: now also J?.4 (Pin_4)
- net LCD_BL: now reaches U?.19 (GPIO14/ADC2_CH3)
- net LCD_BL: now also J?.5 (Pin_5)
- net I2S_DACDAT: now reaches U?.36 (SPICLK_N/GPIO48)
- net I2S_DACDAT: now also U?.10 (DACDAT)
- net I2S_MCK: now reaches U?.37 (SPICLK_P/GPIO47)
- net I2S_MCK: now also U?.11 (MCLK)
- net I2C_SDA: now reaches U?.41 (GPIO36)
- net I2C_SDA: now also U?.17 (SDIN)
- net I2C_SCL: now reaches U?.42 (GPIO37)
- net I2C_SCL: now also U?.16 (SCLK)
- net I2S_LRCK: now reaches U?.43 (GPIO38)
- net I2S_LRCK: now also U?.7 (LRC)
- net I2S_BCLK: now reaches U?.51 (GPIO45)
- net I2S_BCLK: now also U?.8 (BCLK)
- net I2S_ADCDAT: now reaches U?.52 (GPIO46)
- net I2S_ADCDAT: now also U?.9 (ADCDAT)
- net at U?.6 (GPIO1/ADC1_CH0): no longer J?.1 (Pin_1)
- net at U?.7 (GPIO2/ADC1_CH1): no longer J?.2 (Pin_2)
- net at U?.8 (GPIO3/ADC1_CH2): no longer J?.3 (Pin_3)
- net at U?.9 (GPIO4/ADC1_CH3): no longer J?.4 (Pin_4)
- new net: C?.1, C?.2, MK?.4 (OUT)
- new net: C?.2, U?.1 (LIP)
- new net: C?.2, U?.5 (RIN)
- new net: C?.1, U?.27 (VMID)
- new net: C?.1, MK?.1 (VDD), U?.32 (MICBIAS)
- new net: C?.1, R?.2
- new net: C?.2, U?.2 (LIN)
- new net: J?.1 (Pin_1), U?.25 (LOUT2)
- new net: J?.2 (Pin_2), U?.23 (ROUT2)
- new net: C?.2, U?.4 (RIP)
- no-connect marks 6 -> 22
Other:
- moved on the sheet: C?, J?, R?, U?, Y?

Commit message: hw: v1.0
Parts:
- removed J?: Speaker, symbol Connector_Generic:Conn_01x02
- removed J?: (no value), symbol Connector_Generic:Conn_01x08
- removed U?: WM8978, Package_DFN_QFN:QFN-32-1EP_5x5mm_P0.5mm_EP3.3x3.3mm, symbol misc:WM8978
- removed U?: (no value), symbol Regulator_Linear:AMS1117CD-3.3
- added C22, C23: 2.2uf, Capacitor_SMD:C_0402_1005Metric, symbol Device:C
- added C24: 1uf, Capacitor_SMD:C_0402_1005Metric, symbol Device:C
- added J1: TFT_LCD, Connector_FFC-FPC:TE_0-1734839-8_1x08-1MP_P0.5mm_Horizontal, symbol Connector_Generic_MountingPin:Conn_01x08_MountingPin
- added TP7, TP8: TestPoint, TestPoint:TestPoint_Pad_D1.0mm, symbol Connector:TestPoint
- added U1: AMS1117-3.3, Package_TO_SOT_SMD:SOT-223-3_TabPin2, symbol Regulator_Linear:AMS1117-3.3
- added U3: WM8978, Package_DFN_QFN:QFN-32-1EP_5x5mm_P0.5mm_EP3.3x3.3mm, symbol misc:WM8978
- added U4: MPU-6050, Sensor_Motion:InvenSense_QFN-24_4x4mm_P0.5mm, symbol Sensor_Motion:MPU-6050
- AE1: renamed from AE?; value (none) -> Antenna_Shield; footprint (none) -> RF_Antenna:Texas_SWRA117D_2.4GHz_Left
- C1, C4: renamed from C?; value (none) -> 10uf; footprint (none) -> Capacitor_SMD:C_0603_1608Metric
- C10, C13, C14, C15, C16, C18: renamed from C?; value (none) -> 1uf; footprint (none) -> Capacitor_SMD:C_0402_1005Metric
- C11, C12, C9: renamed from C?; value (none) -> 10pf; footprint (none) -> Capacitor_SMD:C_0402_1005Metric
- C17, C19, C20, C21: renamed from C?; value (none) -> 2.2uf; footprint (none) -> Capacitor_SMD:C_0402_1005Metric
- C2: renamed from C?; value (none) -> 1uf; footprint (none) -> Capacitor_SMD:C_0603_1608Metric
- C3, C5, C6: renamed from C?; value (none) -> 0.1uf; footprint (none) -> Capacitor_SMD:C_0402_1005Metric
- C7, C8: renamed from C?; value (none) -> 3pf; footprint (none) -> Capacitor_SMD:C_0402_1005Metric
- J2: renamed from J?; value (none) -> USB_C_Receptacle_USB2.0; footprint (none) -> Connector_USB:USB_C_Receptacle_HRO_TYPE-C-31-M-12
- L1: renamed from L?; value (none) -> 10uh; footprint (none) -> Inductor_SMD:L_0402_1005Metric
- MK1: renamed from MK?; footprint (none) -> misc:MEMS_MIC_2.75x1.85x0.9mm
- R1: renamed from R?; value (none) -> 10k; footprint (none) -> Resistor_SMD:R_0402_1005Metric
- R2, R3: renamed from R?; value (none) -> 5.1k; footprint (none) -> Resistor_SMD:R_0402_1005Metric
- R4: renamed from R?; value (none) -> 0Ω; footprint (none) -> Resistor_SMD:R_0402_1005Metric
- TP1, TP2, TP3, TP4, TP5, TP6: renamed from TP?; value (none) -> TestPoint; footprint (none) -> TestPoint:TestPoint_Pad_D1.0mm
- U2: renamed from U?; value (none) -> ESP32-S3; footprint (none) -> Package_DFN_QFN:QFN-56-1EP_7x7mm_P0.4mm_EP5.6x5.6mm
- Y1: renamed from Y?; value (none) -> 40MHz; footprint (none) -> Crystal:Crystal_SMD_3225-4Pin_3.2x2.5mm
Connections:
- net +3V3: now also C22.2, J1.7 (Pin_7), U1.2 (VO), U3.13 (DCVDD), U3.14 (DBVDD), U3.26 (SPKVDD), U3.31 (AVDD), U4.13 (VDD), U4.8 (VDDIO)
- net +5V: now also J1.8 (Pin_8), U1.3 (VI)
- net GND: now also C22.1, C23.1, C24.1, J1.6 (Pin_6), J1.MP (MountPin), U1.1 (GND), U3.12 (DGND), U3.18 (MODE), U3.24 (SPKGND), U3.28 (AGND), U3.33 (GNDPAD), U4.1 (CLKIN), U4.11 (FSYNC), U4.18 (GND), U4.9 (AD0)
- net I2C_SCL: now also U2.22 (GPIO16/ADC2_CH5/XTAL_32K_N), U3.16 (SCLK), U4.23 (SCL); no longer U2.42 (GPIO37)
- net I2C_SDA: now also U2.23 (GPIO17/ADC2_CH6/DAC_2), U3.17 (SDIN), U4.24 (SDA); no longer U2.41 (GPIO36)
- net I2S_ADCDAT: now also U2.17 (GPIO12/ADC2_CH1), U3.9 (ADCDAT); no longer U2.52 (GPIO46)
- net I2S_BCLK: now also U2.18 (GPIO13/ADC2_CH2), U3.8 (BCLK); no longer U2.51 (GPIO45)
- net I2S_DACDAT: now also U2.16 (GPIO11/ADC2_CH0), U3.10 (DACDAT); no longer U2.36 (SPICLK_N/GPIO48)
- net I2S_LRCK: now also U2.19 (GPIO14/ADC2_CH3), U3.7 (LRC); no longer U2.43 (GPIO38)
- net I2S_MCK: now also U2.15 (GPIO10/ADC1_CH9), U3.11 (MCLK); no longer U2.37 (SPICLK_P/GPIO47)
- net LCD_BL: now also U2.43 (GPIO38), J1.1 (Pin_1); no longer U2.19 (GPIO14/ADC2_CH3)
- net LCD_CS: now also U2.37 (SPICLK_P/GPIO47), J1.2 (Pin_2); no longer U2.17 (GPIO12/ADC2_CH1)
- net LCD_DC: now also U2.24 (GPIO18/ADC2_CH7/DAC_1), J1.5 (Pin_5); no longer U2.18 (GPIO13/ADC2_CH2)
- net LCD_MOSI: now also U2.36 (SPICLK_N/GPIO48), J1.3 (Pin_3); no longer U2.15 (GPIO10/ADC1_CH9)
- net LCD_SCK: now also U2.27 (GPIO21), J1.4 (Pin_4); no longer U2.16 (GPIO11/ADC2_CH0)
- net at C13.2: now also U3.1 (LIP)
- net at C16.2: now also U3.5 (RIN)
- net at C19.1: now also U3.27 (VMID)
- net at C17.1, MK1.1 (VDD): now also U3.32 (MICBIAS)
- net at C14.2: now also U3.2 (LIN)
- net at C15.2: now also U3.4 (RIP)
- new net: TP8.1, U3.23 (ROUT2)
- new net: TP7.1, U3.25 (LOUT2)
- new net: C23.2, U4.20 (CPOUT)
- new net: C24.2, U4.10 (REGOUT)
- no-connect marks 22 -> 42
Other:
- note added: "Internal"
- moved on the sheet: C12, C13, C14, C15, C16, C17, C18, C19, C20, C21, MK1, R4

Commit message: hw: v1.1
Parts:
- added C25: (no value), symbol Device:C
- added C26: 0.1uf, Capacitor_SMD:C_0402_1005Metric, symbol Device:C
- C2: value 1uf -> (none)
- C7, C8: value 3pf -> (none)
- L1: value 10uh -> (none)
Connections:
- net +3V3: now also C25.2, C26.2; no longer C21.2, U3.26 (SPKVDD)
- net +5V: now also C21.2, U3.26 (SPKVDD)
- net GND: now also C25.1, C26.1
Changed lines of the file:
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@@
   (junction (at 50.8 43.18) (diameter 0) (color 0 0 0 0)
   )
+  (junction (at 237.49 21.59) (diameter 0) (color 0 0 0 0)
+  )
   (junction (at 59.69 140.97) (diameter 0) (color 0 0 0 0)
   )
@@
   (junction (at 67.31 30.48) (diameter 0) (color 0 0 0 0)
   )
+  (junction (at 49.53 133.35) (diameter 0) (color 0 0 0 0)
+  )
   (junction (at 50.8 25.4) (diameter 0) (color 0 0 0 0)
   )
@@
   (junction (at 209.55 135.89) (diameter 0) (color 0 0 0 0)
   )
-  (junction (at 240.03 21.59) (diameter 0) (color 0 0 0 0)
-  )
   (junction (at 44.45 179.07) (diameter 0) (color 0 0 0 0)
-  )
-  (junction (at 237.49 21.59) (diameter 0) (color 0 0 0 0)
   )
   (junction (at 151.13 149.86) (diameter 0) (color 0 0 0 0)
@@
     (stroke (width 0) (type default) (color 0 0 0 0))
   )
+  (wire (pts (xy 49.53 140.97) (xy 59.69 140.97))
+    (stroke (width 0) (type default) (color 0 0 0 0))
+  )
   (wire (pts (xy 129.54 30.48) (xy 118.11 30.48))
     (stroke (width 0) (type default) (color 0 0 0 0))
@@
     (stroke (width 0) (type default) (color 0 0 0 0))
   )
-  (wire (pts (xy 49.53 140.97) (xy 59.69 140.97))
-    (stroke (width 0) (type default) (color 0 0 0 0))
-  )
   (wire (pts (xy 237.49 21.59) (xy 237.49 38.1))
     (stroke (width 0) (type default) (color 0 0 0 0))
@@
     (stroke (width 0) (type default) (color 0 0 0 0))
   )
+  (wire (pts (xy 49.53 133.35) (xy 59.69 133.35))
+    (stroke (width 0) (type default) (color 0 0 0 0))
+  )
   (wire (pts (xy 76.2 148.59) (xy 69.85 148.59))
     (stroke (width 0) (type default) (color 0 0 0 0))
@@
   )
   (wire (pts (xy 224.79 81.28) (xy 199.39 81.28))
-    (stroke (width 0) (type default) (color 0 0 0 0))
-  )
-  (wire (pts (xy 224.79 21.59) (xy 237.49 21.59))
     (stroke (width 0) (type default) (color 0 0 0 0))
   )
@@
     (pin "2")
   )
+  (symbol (lib_id "power:+5V") (at 237.49 21.59 0) (unit 1)
+    (in_bom yes) (on_board yes)
+    (property "Reference" "#PWR0141" (id 0) (at 237.49 25.4 0)
+      (effects (font (size 1.27 1.27)) hide)
+    )
+    (property "Value" "+5V" (id 1) (at 236.22 17.78 0)
+      (effects (font (size 1.27 1.27)) (justify left))
+    )
+    (property "Footprint" "" (id 2) (at 237.49 21.59 0)
+      (effects (font (size 1.27 1.27)) hide)
+    )
+    (property "Datasheet" "" (id 3) (at 237.49 21.59 0)
+      (effects (font (size 1.27 1.27)) hide)
+    )
+    (pin "1")
+  )
   (symbol (lib_id "power:GND") (at 67.31 30.48 90) (unit 1)
     (in_bom yes) (on_board yes) (fields_autoplaced)
@@
       (effects (font (size 1.27 1.27)) (justify left))
     )
-    (property "Value" "3pf" (id 1) (at 121.031 28.3722 0)
+    (property "Value" "" (id 1) (at 121.031 28.3722 0)
       (effects (font (size 1.27 1.27)) (justify left))
     )
@@
       (effects (font (size 1.27 1.27)) (justify left))
     )
-    (property "Value" "3pf" (id 1) (at 108.331 28.3722 0)
+    (property "Value" "" (id 1) (at 108.331 28.3722 0)
       (effects (font (size 1.27 1.27)) (justify left))
     )
@@
     (pin "2")
   )
+  (symbol (lib_id "Device:C") (at 59.69 137.16 0) (unit 1)
+    (in_bom yes) (on_board yes) (fields_autoplaced)
+    (property "Reference" "C26" (id 0) (at 62.611 136.3253 0)
+      (effects (font (size 1.27 1.27)) (justify left))
+    )
+    (property "Value" "0.1uf" (id 1) (at 62.611 138.8622 0)
+      (effects (font (size 1.27 1.27)) (justify left))
+    )
+    (property "Footprint" "Capacitor_SMD:C_0402_1005Metric" (id 2) (at 60.6552 140.97 0)
+      (effects (font (size 1.27 1.27)) hide)
+    )
+    (property "Datasheet" "~" (id 3) (at 59.69 137.16 0)
+      (effects (font (size 1.27 1.27)) hide)
+    )
+    (pin "1")
+    (pin "2")
+  )
   (symbol (lib_id "power:GND") (at 59.69 77.47 0) (unit 1)
     (in_bom yes) (on_board yes) (fields_autoplaced)
@@
     (pin "2")
   )
-  (symbol (lib_id "power:+3.3V") (at 240.03 21.59 0) (unit 1)
-    (in_bom yes) (on_board yes)
-    (property "Reference" "#PWR0107" (id 0) (at 240.03 25.4 0)
-      (effects (font (size 1.27 1.27)) hide)
-    )
-    (property "Value" "+3.3V" (id 1) (at 240.03 18.0142 0))
-    (property "Footprint" "" (id 2) (at 240.03 21.59 0)
-      (effects (font (size 1.27 1.27)) hide)
-    )
-    (property "Datasheet" "" (id 3) (at 240.03 21.59 0)
+  (symbol (lib_id "power:+3.3V") (at 224.79 21.59 0) (unit 1)
+    (in_bom yes) (on_board yes)
+    (property "Reference" "#PWR0107" (id 0) (at 224.79 25.4 0)
+      (effects (font (size 1.27 1.27)) hide)
+    )
+    (property "Value" "+3.3V" (id 1) (at 224.79 18.0142 0))
+    (property "Footprint" "" (id 2) (at 224.79 21.59 0)
+      (effects (font (size 1.27 1.27)) hide)
+    )
+    (property "Datasheet" "" (id 3) (at 224.79 21.59 0)
       (effects (font (size 1.27 1.27)) hide)
     )
@@
     )
     (pin "1")
+  )
+  (symbol (lib_id "Device:C") (at 49.53 137.16 0) (unit 1)
+    (in_bom yes) (on_board yes) (fields_autoplaced)
+    (property "Reference" "C25" (id 0) (at 52.451 136.3253 0)
+      (effects (font (size 1.27 1.27)) (justify left))
+    )
+    (property "Value" "" (id 1) (at 52.451 138.8622 0)
+      (effects (font (size 1.27 1.27)) (justify left))
+    )
+    (property "Footprint" "" (id 2) (at 50.4952 140.97 0)
+      (effects (font (size 1.27 1.27)) hide)
+    )
+    (property "Datasheet" "~" (id 3) (at 49.53 137.16 0)
+      (effects (font (size 1.27 1.27)) hide)
+    )
+    (pin "1")
+    (pin "2")
   )
   (symbol (lib_id "power:GND") (at 240.03 29.21 0) (unit 1)
@@
       (effects (font (size 1.27 1.27)) (justify left))
     )
-    (property "Value" "1uf" (id 1) (at 43.561 146.4822 0)
+    (property "Value" "" (id 1) (at 43.561 146.4822 0)
       (effects (font (size 1.27 1.27)) (justify left))
     )
@@
     (in_bom yes) (on_board yes) (fields_autoplaced)
     (property "Reference" "L1" (id 0) (at 111.76 18.6522 90))
-    (property "Value" "10uh" (id 1) (at 111.76 21.1891 90))
+    (property "Value" "" (id 1) (at 111.76 21.1891 90))
     (property "Footprint" "Inductor_SMD:L_0402_1005Metric" (id 2) (at 111.76 22.86 0)
       (effects (font (size 1.27 1.27)) hide)
@@
     (pin "4")
   )
+  (symbol (lib_id "power:GND") (at 49.53 133.35 180) (unit 1)
+    (in_bom yes) (on_board yes) (fields_autoplaced)
+    (property "Reference" "#PWR01" (id 0) (at 49.53 127 0)
+      (effects (font (size 1.27 1.27)) hide)
+    )
+    (property "Value" "GND" (id 1) (at 51.435 132.5138 0)
+      (effects (font (size 1.27 1.27)) (justify right))
+    )
+    (property "Footprint" "" (id 2) (at 49.53 133.35 0)
+      (effects (font (size 1.27 1.27)) hide)
+    )
+    (property "Datasheet" "" (id 3) (at 49.53 133.35 0)
+      (effects (font (size 1.27 1.27)) hide)
+    )
+    (pin "1")
+  )
   (symbol (lib_id "Connector:TestPoint") (at 266.7 49.53 270) (unit 1)
     (in_bom yes) (on_board yes)
@@
       (reference "#FLG0103") (unit 1) (value "PWR_FLAG") (footprint "")
     )
+    (path "/eab031c0-9c3b-48cd-a6db-a44da25a5cc2"
+      (reference "#PWR01") (unit 1) (value "GND") (footprint "")
+    )
     (path "/cc7e536e-3ba7-437a-a3df-f4721f63834d"
       (reference "#PWR0101") (unit 1) (value "GND") (footprint "")
@@
       (reference "#PWR0140") (unit 1) (value "GND") (footprint "")
     )
+    (path "/105f4895-7075-4faf-b842-2988843ccc79"
+      (reference "#PWR0141") (unit 1) (value "+5V") (footprint "")
+    )
     (path "/30821aaa-588b-4bc6-bcef-5bb61fceef3e"
       (reference "AE1") (unit 1) (value "Antenna_Shield") (footprint "RF_Antenna:Texas_SWRA117D_2.4GHz_Left")
@@
     )
     (path "/a144b18a-c204-47f4-b7c4-c46ed75a647d"
-      (reference "C2") (unit 1) (value "1uf") (footprint "Capacitor_SMD:C_0603_1608Metric")
+      (reference "C2") (unit 1) (value "10uf") (footprint "Capacitor_SMD:C_0603_1608Metric")
     )
     (path "/7e9401d8-5e7c-4162-ac40-1a299d7bf70c"
@@
     )
     (path "/2073aaa7-5a88-4ded-9e11-a30d71808468"
-      (reference "C7") (unit 1) (value "3pf") (footprint "Capacitor_SMD:C_0402_1005Metric")
+      (reference "C7") (unit 1) (value "TBD") (footprint "Capacitor_SMD:C_0402_1005Metric")
     )
     (path "/19d68cd5-dc17-40c8-9a91-e755d72c8698"
-      (reference "C8") (unit 1) (value "3pf") (footprint "Capacitor_SMD:C_0402_1005Metric")
+      (reference "C8") (unit 1) (value "TBD") (footprint "Capacitor_SMD:C_0402_1005Metric")
     )
     (path "/4b1d58fe-30e4-4dfe-a71c-70515546f67a"
@@
       (reference "C24") (unit 1) (value "1uf") (footprint "Capacitor_SMD:C_0402_1005Metric")
     )
+    (path "/862163c8-c6df-4776-a3a1-b3662d4f6185"
+      (reference "C25") (unit 1) (value "1uf") (footprint "Capacitor_SMD:C_0402_1005Metric")
+    )
+    (path "/4088e813-1bbe-405d-acc2-03fd4ff3a7ac"
+      (reference "C26") (unit 1) (value "0.1uf") (footprint "Capacitor_SMD:C_0402_1005Metric")
+    )
     (path "/0e282332-42ba-49de-9ba6-00ae7d453029"
       (reference "J1") (unit 1) (value "TFT_LCD") (footprint "Connector_FFC-FPC:TE_0-1734839-8_1x08-1MP_P0.5mm_Horizontal")
@@
     )
     (path "/b339cf93-b5f9-4e58-8f20-b0134d8ed77f"
-      (reference "L1") (unit 1) (value "10uh") (footprint "Inductor_SMD:L_0402_1005Metric")
+      (reference "L1") (unit 1) (value "TBD") (footprint "Inductor_SMD:L_0402_1005Metric")
     )
     (path "/550e8b03-af81-4666-90e0-9af0ab329ea0"
