File: hardware/holocubic.kicad_pcb (KiCad board)
At the start: 2 copper layers, 25.5 x 23.5 mm, 46 parts, among them J1 TFT_LCD, J2 USB_C_Receptacle_USB2.0, U1 AMS1117-3.3, U2 ESP32-S3, U3 WM8978, U4 MPU-6050, Y1 40MHz

Commit message: sw: update
Parts:
- added L1: 10uh, Inductor_SMD:L_0402_1005Metric, F.Cu at (129.9, 104.0)
- moved TP3 1.95 mm to (127.5, 103.2)
- moved C8 1.46 mm to (134.7, 103.5)
- moved L1 1.46 mm to (133.3, 103.1)
- moved C7 0.32 mm to (131.9, 103.5), turned to -90 degrees
- moved C2 0.15 mm to (129.5, 103.0)
Routing:
- net +3V3: track 102.8 -> 57.3 mm, vias 9 -> 13
- net GND: track 41.5 -> 38.3 mm, vias 55 -> 128
- net /LNA: track 2.24 -> 3.64 mm
- net Net-(AE1-Pad1): track 3.94 -> 2.65 mm
- net /I2C_SDA: track 32.0 -> 31.3 mm
- net /I2C_SCL: track 27.9 -> 27.2 mm
- added copper zone on B.Cu, net +3V3
- added copper zone on F.Cu, net +3V3
- added copper zone on In2.Cu, net +3V3
- added copper zone on In1.Cu, net GND
Other:
- copper layers 2 -> 4

Commit message: hw: v1.1
Parts:
- removed the L1 at (129.9, 104.0)
- added C25: 1uf, Capacitor_SMD:C_0402_1005Metric, F.Cu at (129.8, 102.9)
- added C26: 0.1uf, Capacitor_SMD:C_0402_1005Metric, F.Cu at (129.8, 103.6)
- C2: value 1uf -> 10uf; moved to B.Cu
- C7, C8: value 3pf -> TBD
- L1: value 10uh -> TBD
- moved TP5 0.50 mm to (130.8, 104.1)
Connections:
- C21 pad 2: +3V3 -> +5V
- U3 pad 26: +3V3 -> +5V
Routing:
- net +3V3: track 57.3 -> 42.9 mm, vias 13 -> 14
- net +5V: track 31.8 -> 40.0 mm
- net GND: vias 128 -> 134
Other:
- board text added: "HoloCubic-V1.1"
- board text removed: "HoloCubic-V1.0"

Commit message: hw: v1.1
Parts:
- moved TP7 0.35 mm to (133.3, 112.3)
- moved TP8 0.20 mm to (135.0, 112.3)
Other:
- board text added: "SPK"
