File: hardware/main_board/holocubic.kicad_sch (KiCad schematic)
At the start: 48 parts, among them J1 TFT_LCD, J2 USB_C_Receptacle_USB2.0, U1 AMS1117-3.3, U2 ESP32-S3, U3 WM8978, U4 MPU-6050, Y1 40MHz

Commit message: update sch
Parts:
- added L?: 20nH, symbol Device:L
- C2: value (none) -> 10uf
- C25: value (none) -> 1uf; footprint (none) -> Capacitor_SMD:C_0402_1005Metric
- C7, C8, L1: value (none) -> TBD
Connections:
- net at C9.1, Y1.1: now also L?.2; no longer U2.54 (XTAL_P)
- new net: L?.1, U2.54 (XTAL_P)
Changed lines of the file:
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@@
   (junction (at 50.8 43.18) (diameter 0) (color 0 0 0 0)
   )
+  (junction (at 151.13 142.24) (diameter 0) (color 0 0 0 0)
+  )
   (junction (at 237.49 21.59) (diameter 0) (color 0 0 0 0)
   )
@@
   )
   (junction (at 232.41 30.48) (diameter 0) (color 0 0 0 0)
-  )
-  (junction (at 151.13 142.24) (diameter 0) (color 0 0 0 0)
   )
   (junction (at 69.85 138.43) (diameter 0) (color 0 0 0 0)
@@
     (stroke (width 0) (type default) (color 0 0 0 0))
   )
+  (wire (pts (xy 138.43 142.24) (xy 139.7 142.24))
+    (stroke (width 0) (type default) (color 0 0 0 0))
+  )
   (wire (pts (xy 200.66 120.65) (xy 209.55 120.65))
     (stroke (width 0) (type default) (color 0 0 0 0))
@@
     (stroke (width 0) (type default) (color 0 0 0 0))
   )
+  (wire (pts (xy 147.32 142.24) (xy 151.13 142.24))
+    (stroke (width 0) (type default) (color 0 0 0 0))
+  )
   (wire (pts (xy 151.13 149.86) (xy 166.37 149.86))
     (stroke (width 0) (type default) (color 0 0 0 0))
@@
   )
   (wire (pts (xy 185.42 44.45) (xy 185.42 46.99))
-    (stroke (width 0) (type default) (color 0 0 0 0))
-  )
-  (wire (pts (xy 138.43 142.24) (xy 151.13 142.24))
     (stroke (width 0) (type default) (color 0 0 0 0))
   )
@@
     (pin "1")
   )
+  (symbol (lib_id "Device:L") (at 143.51 142.24 90) (unit 1)
+    (in_bom yes) (on_board yes)
+    (property "Reference" "L?" (id 0) (at 146.05 143.51 90))
+    (property "Value" "20nH" (id 1) (at 140.97 143.51 90))
+    (property "Footprint" "" (id 2) (at 143.51 142.24 0)
+      (effects (font (size 1.27 1.27)) hide)
+    )
+    (property "Datasheet" "~" (id 3) (at 143.51 142.24 0)
+      (effects (font (size 1.27 1.27)) hide)
+    )
+    (pin "1")
+    (pin "2")
+  )
   (symbol (lib_id "power:GND") (at 67.31 30.48 90) (unit 1)
     (in_bom yes) (on_board yes) (fields_autoplaced)
@@
       (effects (font (size 1.27 1.27)) (justify left))
     )
-    (property "Value" "" (id 1) (at 121.031 28.3722 0)
+    (property "Value" "TBD" (id 1) (at 121.031 28.3722 0)
       (effects (font (size 1.27 1.27)) (justify left))
     )
@@
       (effects (font (size 1.27 1.27)) (justify left))
     )
-    (property "Value" "" (id 1) (at 108.331 28.3722 0)
+    (property "Value" "TBD" (id 1) (at 108.331 28.3722 0)
       (effects (font (size 1.27 1.27)) (justify left))
     )
@@
       (effects (font (size 1.27 1.27)) (justify left))
     )
-    (property "Value" "" (id 1) (at 52.451 138.8622 0)
-      (effects (font (size 1.27 1.27)) (justify left))
-    )
-    (property "Footprint" "" (id 2) (at 50.4952 140.97 0)
+    (property "Value" "1uf" (id 1) (at 52.451 138.8622 0)
+      (effects (font (size 1.27 1.27)) (justify left))
+    )
+    (property "Footprint" "Capacitor_SMD:C_0402_1005Metric" (id 2) (at 50.4952 140.97 0)
       (effects (font (size 1.27 1.27)) hide)
     )
@@
       (effects (font (size 1.27 1.27)) (justify left))
     )
-    (property "Value" "" (id 1) (at 43.561 146.4822 0)
+    (property "Value" "10uf" (id 1) (at 43.561 146.4822 0)
       (effects (font (size 1.27 1.27)) (justify left))
     )
@@
     (in_bom yes) (on_board yes) (fields_autoplaced)
     (property "Reference" "L1" (id 0) (at 111.76 18.6522 90))
-    (property "Value" "" (id 1) (at 111.76 21.1891 90))
+    (property "Value" "TBD" (id 1) (at 111.76 21.1891 90))
     (property "Footprint" "Inductor_SMD:L_0402_1005Metric" (id 2) (at 111.76 22.86 0)
       (effects (font (size 1.27 1.27)) hide)
@@
       (reference "L1") (unit 1) (value "TBD") (footprint "Inductor_SMD:L_0402_1005Metric")
     )
+    (path "/15b79e49-cde0-45d8-ad6d-913a1dbd72f0"
+      (reference "L?") (unit 1) (value "20nH") (footprint "")
+    )
     (path "/550e8b03-af81-4666-90e0-9af0ab329ea0"
